File: PCB/flyback/flyback.kicad_sch (KiCad schematic)
At the start: 7 parts, among them T1 Transformer_1P_1S

Commit message: Schematic Update
Parts:
- removed D?: MM3Zxx, Diode_SMD:D_SOD-323F, symbol Diode:MM3Zxx
- added C? (x16): C, symbol Device:C
- added D?: 1N4002, Diode_THT:D_DO-41_SOD81_P10.16mm_Horizontal, symbol Diode:1N4002
- added D?: MBR735, Package_TO_SOT_THT:TO-220-2_Vertical, symbol Diode:MBR735
- added R? (x15): R, symbol Device:R
Connections:
- net at Q?.1 (G): now also R?.2
- net at Q?.2 (D): now also T1.2 (AB), D?.2 (A)
- net at U?.1: now also R?.2
- net at U?.2: now also U?.1 (K), R?.1, R?.2
- net at U?.4: now also R?.1
- net at U?.1 (COMP): now also C?.2, R?.2
- net at U?.3 (CS): now also C?.2
- net at U?.4 (RC): now also C?.1, R?.2
- net at U?.6 (OUT): now also R?.1
- net at U?.7 (VCC): now also C?.2, C?.2, C?.2
- net at U?.8 (VREF): now also C?.1, R?.1
- net at T1.1 (AA): now also C?.2, C?.2, C?.2
- net at T1.3 (SA): now also C?.1, C?.1, C?.1
- net at T1.4 (SB): now also D?.2 (A), R?.1
- net at U?.2 (REF): now also C?.2, R?.1
- net at D?.1 (K): now also R?.1, R?.2
- new net: C?.1, R?.2 (x2)
- new net: C?.1, R?.1, R?.2
- new net: R?.1, R?.2, R?.2
- new net: C?.1, R?.1, R?.1
- new net: C?.2, D?.1 (K), R?.2, R?.2
- new net Vout: C?.2, C?.2, C?.2, C?.2, D?.1 (K), R?.1, R?.1, R?.1
Other:
- moved on the sheet: D?, Q?, U?

Commit message: Schematic Update
Parts:
- added R? (x3): R, symbol Device:R
Connections:
- net Vfb: now reaches R?.1
- net Vfb: now also R?.1, U?.4
- net GNDA: now reaches R?.2
- net GNDA: now also C?.1, C?.1, C?.1, C?.1, C?.1, C?.1, C?.1, C?.2, C?.2, D?.2 (A), R?.2, T1.3 (SA), U?.3 (A), U?.5 (GND), R?.2, R?.2, R?.2
- net at C?.2, C?.2, C?.2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: now also C?.1, R?.1
- net at Q?.3 (S): now also R?.1, R?.1, R?.1
- net Vref: now reaches C?.1, R?.1, U?.8 (VREF)
- net Vref: now also U?.5
- now unconnected: R?.1

Commit message: Flyback Update
Parts:
- added C?: C, symbol Device:C
- added R?: 47, Resistor_SMD:R_0805_2012Metric, symbol Device:R
- C?: value C -> 100n; footprint (none) -> Capacitor_SMD:C_0805_2012Metric
- C? (x2): value C -> 1u; footprint (none) -> Capacitor_SMD:C_0805_2012Metric
- C?: value C -> 10n; footprint (none) -> Capacitor_SMD:C_0805_2012Metric
- R?: value R -> 820k; footprint (none) -> Resistor_SMD:R_0805_2012Metric
- R?: value R -> 10; footprint (none) -> Resistor_SMD:R_0805_2012Metric
- R?: value R -> 4.7k; footprint (none) -> Resistor_SMD:R_0805_2012Metric
- R? (x3): value R -> 10k; footprint (none) -> Resistor_SMD:R_0805_2012Metric
- R? (x3): value R -> 1k; footprint (none) -> Resistor_SMD:R_0805_2012Metric
- R? (x3): value R -> 22k; footprint (none) -> Resistor_SMD:R_0805_2012Metric
- R?: value R -> 12k; footprint (none) -> Resistor_SMD:R_0805_2012Metric
- R? (x3): value R -> 150m; footprint (none) -> Resistor_SMD:R_2512_6332Metric
- R?: value R -> 182k; footprint (none) -> Resistor_SMD:R_0805_2012Metric
- R?: value R -> 100; footprint (none) -> Resistor_SMD:R_0805_2012Metric
Connections:
- net GNDA: now also C?.1, C?.1, C?.1
- net at D?.2 (A), Q?.2 (D), T1.2 (AB): now also R?.1
- net at Q?.3 (S), R?.1, R?.1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: now also C?.1
- new net: C?.2, R?.2
Other:
- moved on the sheet: R?

Commit message: Schematic Finalize
Parts:
- removed C? (x3): C, symbol Device:C
- added C15, C16, C17: 10u, Capacitor_SMD:C_2220_5650Metric, symbol Device:C
- added C18: 4.7u, Capacitor_SMD:C_2220_5650Metric, symbol Device:C
- added C5: 100n, Capacitor_SMD:C_0805_2012Metric, symbol Device:C
- added C7: 10n, Capacitor_SMD:C_1206_3216Metric, symbol Device:C
- C10: renamed from C?; value C -> 220n; footprint (none) -> Capacitor_SMD:C_0805_2012Metric
- C11: renamed from C?; value C -> 4.7n; footprint (none) -> Capacitor_SMD:C_0805_2012Metric
- C12: renamed from C?; value C -> 470p; footprint (none) -> Capacitor_SMD:C_1206_3216Metric
- C13: renamed from C?; value C -> 10u; footprint (none) -> Capacitor_SMD:C_2220_5650Metric
- C14: renamed from C?; value C -> 1n; footprint (none) -> Capacitor_SMD:C_0805_2012Metric
- C19: renamed from C?; value C -> 100n; footprint (none) -> Capacitor_SMD:C_0805_2012Metric
- C2: renamed from C?; value C -> 100p; footprint (none) -> Capacitor_SMD:C_0805_2012Metric
- C20: renamed from C?; value C -> 10n; footprint (none) -> Capacitor_SMD:C_1206_3216Metric
- C3: renamed from C?; value C -> 2.2n; footprint (none) -> Capacitor_SMD:C_0805_2012Metric
- C8: renamed from C?; footprint Capacitor_SMD:C_0805_2012Metric -> Capacitor_SMD:C_1206_3216Metric
- C9: renamed from C?; value C -> 0.47n; footprint (none) -> Capacitor_SMD:C_0805_2012Metric
- D2: renamed from D?; value MBR735 -> MBR10150
- D3: renamed from D?; value MMSD4148 -> MMSZ4713
- Q1: renamed from Q?; value QM6006D -> IRFR3410TRLPBF
- gave numbers to parts that had none: 26
Connections:
- net GNDA: now also C15.1, C16.1, C17.1, C18.1, C5.1, C7.1
- net Vout: now also C15.2, C16.2, C17.2, C18.2
- net at U1.7 (VCC): now also C10.1, C4.2, C6.2, C8.2, R4.1, T1.1 (AA), C5.2, C7.2
Other:
- moved on the sheet: C19, C20

Commit message: PCB Update
Parts:
- T1: footprint Transformer_THT:Transformer_CHK_EI42-5VA_Neutral -> Transformer_THT:Transformer_CHK_EI48-10VA_Neutral
Connections:
- net GNDA: now also T1.10 (SA); no longer T1.3 (SA)
- net at C2.1, R1.2, R2.1: now also U1.2 (FB)
- net at C10.1, C4.2, C5.2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: now also T1.5 (AA); no longer T1.1 (AA)
- net at D1.2 (A), Q1.2 (D), R10.1: now also T1.1 (AB); no longer T1.2 (AB)
- net at D2.2 (A), R12.1: now also T1.6 (SB); no longer T1.4 (SB)
Changed lines of the file:
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@@
   (junction (at 102.87 67.056) (diameter 0) (color 0 0 0 0)
   )
+  (junction (at 59.436 81.661) (diameter 0) (color 0 0 0 0)
+  )
   (junction (at 197.104 89.281) (diameter 0) (color 0 0 0 0)
   )
@@
     (stroke (width 0) (type default) (color 0 0 0 0))
   )
+  (wire (pts (xy 90.17 88.392) (xy 90.17 87.757))
+    (stroke (width 0) (type default) (color 0 0 0 0))
+  )
   (wire (pts (xy 88.646 56.134) (xy 88.646 56.261))
     (stroke (width 0) (type default) (color 0 0 0 0))
@@
     (stroke (width 0) (type default) (color 0 0 0 0))
   )
+  (wire (pts (xy 59.436 81.661) (xy 60.706 81.661))
+    (stroke (width 0) (type default) (color 0 0 0 0))
+  )
   (wire (pts (xy 74.549 89.027) (xy 74.549 90.805))
     (stroke (width 0) (type default) (color 0 0 0 0))
@@
     (stroke (width 0) (type default) (color 0 0 0 0))
   )
+  (wire (pts (xy 59.436 88.392) (xy 59.436 81.661))
+    (stroke (width 0) (type default) (color 0 0 0 0))
+  )
   (wire (pts (xy 187.198 78.232) (xy 197.104 78.232))
     (stroke (width 0) (type default) (color 0 0 0 0))
@@
     (stroke (width 0) (type default) (color 0 0 0 0))
   )
+  (wire (pts (xy 90.17 88.392) (xy 59.436 88.392))
+    (stroke (width 0) (type default) (color 0 0 0 0))
+  )
   (wire (pts (xy 197.104 89.281) (xy 204.597 89.281))
     (stroke (width 0) (type default) (color 0 0 0 0))
@@
     (stroke (width 0) (type default) (color 0 0 0 0))
   )
-  (wire (pts (xy 58.547 81.661) (xy 60.706 81.661))
+  (wire (pts (xy 58.547 81.661) (xy 59.436 81.661))
     (stroke (width 0) (type default) (color 0 0 0 0))
   )
@@
     (property "Reference" "T1" (id 0) (at 157.8737 52.07 0))
     (property "Value" "Transformer_1P_1S" (id 1) (at 157.8737 54.61 0))
-    (property "Footprint" "Transformer_THT:Transformer_CHK_EI42-5VA_Neutral" (id 2) (at 157.861 61.722 0)
+    (property "Footprint" "Transformer_THT:Transformer_CHK_EI48-10VA_Neutral" (id 2) (at 157.861 61.722 0)
       (effects (font (size 1.27 1.27)) hide)
     )
@@
     )
     (pin "1")
-    (pin "2")
-    (pin "3")
-    (pin "4")
+    (pin "10")
+    (pin "5")
+    (pin "6")
   )
   (symbol (lib_id "Device:R") (at 108.839 60.198 0) (unit 1)
@@
     )
     (path "/b5d01af5-8ae7-44b6-90bf-a36ba0c75834"
-      (reference "T1") (unit 1) (value "Transformer_1P_1S") (footprint "Transformer_THT:Transformer_CHK_EI42-5VA_Neutral")
+      (reference "T1") (unit 1) (value "Transformer_1P_1S") (footprint "Transformer_THT:Transformer_CHK_EI48-10VA_Neutral")
     )
     (path "/ab106f85-0f50-4e3d-a047-d2875db758ad"

Commit message: Layout Update
Connections:
- net GNDA: no longer C1.2, C13.1, C15.1, C16.1, C17.1, C18.1, C19.1, C20.1, C3.2, C4.1, C5.1, C6.1, C7.1, C8.1, C9.1, R19.2, R7.2, R8.2, R9.2, T1.10 (SA), U1.5 (GND), U3.3 (A)
- new net GND1: C1.2, C3.2, C4.1, C5.1, C6.1, C8.1, C9.1, R7.2, R8.2, R9.2, U1.5 (GND)
- new net GND2: C13.1, C15.1, C16.1, C17.1, C18.1, C19.1, C20.1, R19.2, T1.10 (SA), U3.3 (A)

Commit message: PCB Update
Parts:
- added R20: 10k, Resistor_SMD:R_0805_2012Metric, symbol Device:R
- T1: footprint Transformer_THT:Transformer_CHK_EI48-10VA_Neutral -> Transformer_THT:Transformer_CHK_EI48-8VA_Neutral
Connections:
- net GND1: now also R20.1
- net GND2: now also T1.12 (SA); no longer T1.10 (SA)
- net at Q1.1 (G), R6.2: now also R20.2
- net Vin: now reaches C10.1, C4.2, C5.2, C6.2, C7.2, C8.2, R4.1, U1.7 (VCC)
- net Vin: now also R5.1, T1.6 (AA); no longer T1.5 (AA)
- net at D2.2 (A), R12.1: now also T1.7 (SB); no longer T1.6 (SB)

Commit message: PCB Update
Connections:
- net GND1: now also C7.1
- net GND2: now also D3.2 (A)
- net GNDA: no longer D3.2 (A)
Changed lines of the file:
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@@
   (junction (at 79.375 47.244) (diameter 0) (color 0 0 0 0)
   )
-  (junction (at 87.884 75.057) (diameter 0) (color 0 0 0 0)
-  )
   (junction (at 144.018 108.204) (diameter 0) (color 0 0 0 0)
   )
@@
   (junction (at 202.438 48.387) (diameter 0) (color 0 0 0 0)
   )
+  (junction (at 87.884 75.184) (diameter 0) (color 0 0 0 0)
+  )
   (junction (at 227.076 66.802) (diameter 0) (color 0 0 0 0)
   )
@@
     (stroke (width 0) (type default) (color 0 0 0 0))
   )
+  (wire (pts (xy 96.52 74.676) (xy 96.52 75.184))
+    (stroke (width 0) (type default) (color 0 0 0 0))
+  )
   (wire (pts (xy 161.036 110.49) (xy 167.767 110.49))
     (stroke (width 0) (type default) (color 0 0 0 0))
@@
     (stroke (width 0) (type default) (color 0 0 0 0))
   )
-  (wire (pts (xy 87.884 75.057) (xy 87.884 75.692))
+  (wire (pts (xy 87.884 75.057) (xy 87.884 75.184))
     (stroke (width 0) (type default) (color 0 0 0 0))
   )
@@
     (stroke (width 0) (type default) (color 0 0 0 0))
   )
-  (wire (pts (xy 204.597 96.901) (xy 204.597 97.79))
+  (wire (pts (xy 204.597 96.901) (xy 204.597 98.679))
     (stroke (width 0) (type default) (color 0 0 0 0))
   )
@@
     (stroke (width 0) (type default) (color 0 0 0 0))
   )
+  (wire (pts (xy 87.884 75.184) (xy 87.884 75.692))
+    (stroke (width 0) (type default) (color 0 0 0 0))
+  )
   (wire (pts (xy 225.044 115.951) (xy 230.886 115.951))
     (stroke (width 0) (type default) (color 0 0 0 0))
@@
     (stroke (width 0) (type default) (color 0 0 0 0))
   )
-  (wire (pts (xy 96.52 75.184) (xy 87.884 75.184))
-    (stroke (width 0) (type default) (color 0 0 0 0))
-  )
   (wire (pts (xy 144.399 119.761) (xy 144.399 121.285))
     (stroke (width 0) (type default) (color 0 0 0 0))
@@
     (stroke (width 0) (type default) (color 0 0 0 0))
   )
-  (wire (pts (xy 96.52 74.676) (xy 96.52 75.184))
+  (wire (pts (xy 87.884 75.184) (xy 96.52 75.184))
     (stroke (width 0) (type default) (color 0 0 0 0))
   )
@@
   (label "Vfb" (at 48.133 81.661 0)
     (effects (font (size 1.27 1.27)) (justify left bottom))
-  )
-  (symbol (lib_id "power:GNDA") (at 204.597 97.79 0) (unit 1)
-    (in_bom yes) (on_board yes) (fields_autoplaced)
-    (property "Reference" "#PWR010" (id 0) (at 204.597 104.14 0)
-      (effects (font (size 1.27 1.27)) hide)
-    )
-    (property "Value" "GNDA" (id 1) (at 204.597 103.251 0))
-    (property "Footprint" "" (id 2) (at 204.597 97.79 0)
-      (effects (font (size 1.27 1.27)) hide)
-    )
-    (property "Datasheet" "" (id 3) (at 204.597 97.79 0)
-      (effects (font (size 1.27 1.27)) hide)
-    )
-    (pin "1")
   )
   (symbol (lib_id "power:GND1") (at 52.451 99.822 0) (unit 1)
@@
     (pin "1")
     (pin "2")
+  )
+  (symbol (lib_id "power:GND2") (at 204.597 98.679 0) (unit 1)
+    (in_bom yes) (on_board yes) (fields_autoplaced)
+    (property "Reference" "#PWR?" (id 0) (at 204.597 105.029 0)
+      (effects (font (size 1.27 1.27)) hide)
+    )
+    (property "Value" "GND2" (id 1) (at 204.597 103.124 0))
+    (property "Footprint" "" (id 2) (at 204.597 98.679 0)
+      (effects (font (size 1.27 1.27)) hide)
+    )
+    (property "Datasheet" "" (id 3) (at 204.597 98.679 0)
+      (effects (font (size 1.27 1.27)) hide)
+    )
+    (pin "1")
   )
   (symbol (lib_id "Transistor_FET:QM6006D") (at 141.478 85.217 0) (unit 1)
@@
       (reference "#PWR08") (unit 1) (value "GNDA") (footprint "")
     )
-    (path "/028d1225-17b1-4284-b8ae-c061c4274de5"
-      (reference "#PWR010") (unit 1) (value "GNDA") (footprint "")
-    )
     (path "/3195101c-5fa3-454b-9b48-ae328327334f"
       (reference "#PWR0101") (unit 1) (value "GND1") (footprint "")
@@
       (reference "#PWR0110") (unit 1) (value "GND2") (footprint "")
     )
+    (path "/2f535012-90dd-40a5-adee-4a63a2d8ccfa"
+      (reference "#PWR?") (unit 1) (value "GND2") (footprint "")
+    )
     (path "/8120bd45-6ae9-4b9f-bc73-a930ab5f2dd6"
