File: PCB/flyback/flyback.kicad_sch (KiCad schematic)
At the start: 48 parts, among them Q1 IRFR3410TRLPBF, T1 Transformer_1P_1S, U1 UC3843_SOIC8, U2 4N25, U3 TL431DBZ

Commit message: Schematic Update
Parts:
- added H1, H2, H3, H4: MountingHole_Pad, MountingHole:MountingHole_2.2mm_M2, symbol Mechanical:MountingHole_Pad
Connections:
- net GND1: now also H1.1
- net GND2: now also H4.1
- net Vin: now also H2.1
- net Vout: now also H3.1
Changed lines of the file:
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@@
   (junction (at 214.249 66.802) (diameter 0) (color 0 0 0 0)
   )
+  (junction (at 88.646 57.15) (diameter 0) (color 0 0 0 0)
+  )
   (junction (at 197.104 78.232) (diameter 0) (color 0 0 0 0)
   )
@@
     (stroke (width 0) (type default) (color 0 0 0 0))
   )
+  (wire (pts (xy 53.213 57.15) (xy 88.646 57.15))
+    (stroke (width 0) (type default) (color 0 0 0 0))
+  )
   (wire (pts (xy 139.827 56.642) (xy 139.827 47.244))
     (stroke (width 0) (type default) (color 0 0 0 0))
@@
     (stroke (width 0) (type default) (color 0 0 0 0))
   )
+  (wire (pts (xy 256.667 45.593) (xy 256.667 48.387))
+    (stroke (width 0) (type default) (color 0 0 0 0))
+  )
   (wire (pts (xy 117.348 63.754) (xy 117.348 66.802))
     (stroke (width 0) (type default) (color 0 0 0 0))
@@
     (stroke (width 0) (type default) (color 0 0 0 0))
   )
-  (wire (pts (xy 79.375 46.609) (xy 79.375 47.244))
+  (wire (pts (xy 79.375 43.18) (xy 79.375 47.244))
     (stroke (width 0) (type default) (color 0 0 0 0))
   )
@@
     (stroke (width 0) (type default) (color 0 0 0 0))
   )
-  (wire (pts (xy 249.555 48.387) (xy 250.317 48.387))
+  (wire (pts (xy 249.555 48.387) (xy 256.667 48.387))
     (stroke (width 0) (type default) (color 0 0 0 0))
   )
@@
     (stroke (width 0) (type default) (color 0 0 0 0))
   )
+  (wire (pts (xy 53.213 54.102) (xy 53.213 57.15))
+    (stroke (width 0) (type default) (color 0 0 0 0))
+  )
   (wire (pts (xy 144.018 90.297) (xy 144.018 94.107))
     (stroke (width 0) (type default) (color 0 0 0 0))
@@
     (stroke (width 0) (type default) (color 0 0 0 0))
   )
+  (wire (pts (xy 259.588 64.008) (xy 259.588 65.278))
+    (stroke (width 0) (type default) (color 0 0 0 0))
+  )
   (wire (pts (xy 87.884 75.184) (xy 96.52 75.184))
     (stroke (width 0) (type default) (color 0 0 0 0))
@@
     (stroke (width 0) (type default) (color 0 0 0 0))
   )
-  (wire (pts (xy 88.646 56.261) (xy 88.646 57.531))
+  (wire (pts (xy 88.646 56.261) (xy 88.646 57.15))
     (stroke (width 0) (type default) (color 0 0 0 0))
   )
@@
   )
   (wire (pts (xy 186.055 48.387) (xy 191.389 48.387))
+    (stroke (width 0) (type default) (color 0 0 0 0))
+  )
+  (wire (pts (xy 88.646 57.15) (xy 88.646 57.531))
     (stroke (width 0) (type default) (color 0 0 0 0))
   )
@@
   (symbol (lib_id "power:GND2") (at 204.597 98.679 0) (unit 1)
     (in_bom yes) (on_board yes) (fields_autoplaced)
-    (property "Reference" "#PWR?" (id 0) (at 204.597 105.029 0)
+    (property "Reference" "#PWR0111" (id 0) (at 204.597 105.029 0)
       (effects (font (size 1.27 1.27)) hide)
     )
@@
     (pin "1")
   )
+  (symbol (lib_id "Mechanical:MountingHole_Pad") (at 53.213 51.562 0) (unit 1)
+    (in_bom yes) (on_board yes) (fields_autoplaced)
+    (property "Reference" "H1" (id 0) (at 56.134 49.0219 0)
+      (effects (font (size 1.27 1.27)) (justify left))
+    )
+    (property "Value" "MountingHole_Pad" (id 1) (at 56.134 51.5619 0)
+      (effects (font (size 1.27 1.27)) (justify left))
+    )
+    (property "Footprint" "MountingHole:MountingHole_2.2mm_M2" (id 2) (at 53.213 51.562 0)
+      (effects (font (size 1.27 1.27)) hide)
+    )
+    (property "Datasheet" "~" (id 3) (at 53.213 51.562 0)
+      (effects (font (size 1.27 1.27)) hide)
+    )
+    (pin "1")
+  )
   (symbol (lib_id "Device:R") (at 161.036 118.618 0) (unit 1)
     (in_bom yes) (on_board yes) (fields_autoplaced)
@@
     (pin "2")
   )
+  (symbol (lib_id "Mechanical:MountingHole_Pad") (at 256.667 43.053 0) (unit 1)
+    (in_bom yes) (on_board yes) (fields_autoplaced)
+    (property "Reference" "H3" (id 0) (at 259.588 40.5129 0)
+      (effects (font (size 1.27 1.27)) (justify left))
+    )
+    (property "Value" "MountingHole_Pad" (id 1) (at 259.588 43.0529 0)
+      (effects (font (size 1.27 1.27)) (justify left))
+    )
+    (property "Footprint" "MountingHole:MountingHole_2.2mm_M2" (id 2) (at 256.667 43.053 0)
+      (effects (font (size 1.27 1.27)) hide)
+    )
+    (property "Datasheet" "~" (id 3) (at 256.667 43.053 0)
+      (effects (font (size 1.27 1.27)) hide)
+    )
+    (pin "1")
+  )
   (symbol (lib_id "Device:R") (at 74.549 94.615 0) (unit 1)
     (in_bom yes) (on_board yes) (fields_autoplaced)
@@
     (pin "1")
     (pin "2")
+  )
+  (symbol (lib_id "Mechanical:MountingHole_Pad") (at 259.588 61.468 0) (unit 1)
+    (in_bom yes) (on_board yes) (fields_autoplaced)
+    (property "Reference" "H4" (id 0) (at 262.509 58.9279 0)
+      (effects (font (size 1.27 1.27)) (justify left))
+    )
+    (property "Value" "MountingHole_Pad" (id 1) (at 262.509 61.4679 0)
+      (effects (font (size 1.27 1.27)) (justify left))
+    )
+    (property "Footprint" "MountingHole:MountingHole_2.2mm_M2" (id 2) (at 259.588 61.468 0)
+      (effects (font (size 1.27 1.27)) hide)
+    )
+    (property "Datasheet" "~" (id 3) (at 259.588 61.468 0)
+      (effects (font (size 1.27 1.27)) hide)
+    )
+    (pin "1")
   )
   (symbol (lib_id "Device:C") (at 52.451 94.742 0) (unit 1)
@@
     (pin "1")
     (pin "2")
+  )
+  (symbol (lib_id "power:GND2") (at 259.588 65.278 0) (unit 1)
+    (in_bom yes) (on_board yes) (fields_autoplaced)
+    (property "Reference" "#PWR01" (id 0) (at 259.588 71.628 0)
+      (effects (font (size 1.27 1.27)) hide)
+    )
+    (property "Value" "GND2" (id 1) (at 259.588 69.723 0))
+    (property "Footprint" "" (id 2) (at 259.588 65.278 0)
+      (effects (font (size 1.27 1.27)) hide)
+    )
+    (property "Datasheet" "" (id 3) (at 259.588 65.278 0)
+      (effects (font (size 1.27 1.27)) hide)
+    )
+    (pin "1")
   )
   (symbol (lib_id "Diode:1N4002") (at 135.128 66.802 0) (unit 1)
@@
     (pin "5")
     (pin "6")
+  )
+  (symbol (lib_id "Mechanical:MountingHole_Pad") (at 79.375 40.64 0) (unit 1)
+    (in_bom yes) (on_board yes) (fields_autoplaced)
+    (property "Reference" "H2" (id 0) (at 82.296 38.0999 0)
+      (effects (font (size 1.27 1.27)) (justify left))
+    )
+    (property "Value" "MountingHole_Pad" (id 1) (at 82.296 40.6399 0)
+      (effects (font (size 1.27 1.27)) (justify left))
+    )
+    (property "Footprint" "MountingHole:MountingHole_2.2mm_M2" (id 2) (at 79.375 40.64 0)
+      (effects (font (size 1.27 1.27)) hide)
+    )
+    (property "Datasheet" "~" (id 3) (at 79.375 40.64 0)
+      (effects (font (size 1.27 1.27)) hide)
+    )
+    (pin "1")
   )
   (symbol (lib_id "Device:C") (at 128.524 60.071 0) (unit 1)
@@
   )
   (symbol_instances
+    (path "/93bed2a4-4513-41ed-852b-819e1c15c6db"
+      (reference "#PWR01") (unit 1) (value "GND2") (footprint "")
+    )
     (path "/594f1f93-70f8-479e-ab33-5d76880075fc"
       (reference "#PWR08") (unit 1) (value "GNDA") (footprint "")
@@
     )
     (path "/2f535012-90dd-40a5-adee-4a63a2d8ccfa"
-      (reference "#PWR?") (unit 1) (value "GND2") (footprint "")
+      (reference "#PWR0111") (unit 1) (value "GND2") (footprint "")
     )
     (path "/8120bd45-6ae9-4b9f-bc73-a930ab5f2dd6"
@@
       (reference "D3") (unit 1) (value "MMSZ4713") (footprint "Diode_SMD:D_SOD-123")
     )
+    (path "/56db1a75-0d4f-4784-9097-648cacbc63d5"
+      (reference "H1") (unit 1) (value "MountingHole_Pad") (footprint "MountingHole:MountingHole_2.2mm_M2")
+    )
+    (path "/9da11739-fb10-4b57-8e97-6da8c7049905"
+      (reference "H2") (unit 1) (value "MountingHole_Pad") (footprint "MountingHole:MountingHole_2.2mm_M2")
+    )
+    (path "/75f27a60-8b14-41a7-aa57-892b186f726b"
+      (reference "H3") (unit 1) (value "MountingHole_Pad") (footprint "MountingHole:MountingHole_2.2mm_M2")
+    )
+    (path "/7da4b92f-21e1-4f36-9906-cc49f0feb7b8"
+      (reference "H4") (unit 1) (value "MountingHole_Pad") (footprint "MountingHole:MountingHole_2.2mm_M2")
+    )
     (path "/30378621-bd04-41ec-aa0e-44428c384fa5"

Commit message: Transformer Footprint Updated
Parts:
- T1: footprint Transformer_THT:Transformer_CHK_EI48-8VA_Neutral -> Transformer_THT:Transformer_37x44
Changed lines of the file:
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@@
     (property "Reference" "T1" (id 0) (at 157.8737 52.07 0))
     (property "Value" "Transformer_1P_1S" (id 1) (at 157.8737 54.61 0))
-    (property "Footprint" "Transformer_THT:Transformer_CHK_EI48-8VA_Neutral" (id 2) (at 157.861 61.722 0)
+    (property "Footprint" "Transformer_THT:Transformer_37x44" (id 2) (at 157.861 61.722 0)
       (effects (font (size 1.27 1.27)) hide)
     )
@@
     )
     (path "/b5d01af5-8ae7-44b6-90bf-a36ba0c75834"
-      (reference "T1") (unit 1) (value "Transformer_1P_1S") (footprint "Transformer_THT:Transformer_CHK_EI48-8VA_Neutral")
+      (reference "T1") (unit 1) (value "Transformer_1P_1S") (footprint "Transformer_THT:Transformer_37x44")
     )
     (path "/ab106f85-0f50-4e3d-a047-d2875db758ad"

Commit message: V3_flyback
Parts:
- U2: footprint Package_DIP:DIP-6_W7.62mm -> Package_DIP:DIP-6_W7.62mm_SMDSocket_SmallPads
Changed lines of the file:
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@@
   (junction (at 144.399 119.761) (diameter 0) (color 0 0 0 0)
   )
+  (junction (at 60.706 81.661) (diameter 0) (color 0 0 0 0)
+  )
+  (junction (at 74.549 89.027) (diameter 0) (color 0 0 0 0)
+  )
+  (junction (at 88.646 56.134) (diameter 0) (color 0 0 0 0)
+  )
+  (junction (at 220.726 48.387) (diameter 0) (color 0 0 0 0)
+  )
+  (junction (at 189.611 113.03) (diameter 0) (color 0 0 0 0)
+  )
+  (junction (at 249.555 48.387) (diameter 0) (color 0 0 0 0)
+  )
+  (junction (at 88.646 47.244) (diameter 0) (color 0 0 0 0)
+  )
+  (junction (at 240.919 66.802) (diameter 0) (color 0 0 0 0)
+  )
+  (junction (at 128.524 66.802) (diameter 0) (color 0 0 0 0)
+  )
+  (junction (at 74.549 99.314) (diameter 0) (color 0 0 0 0)
+  )
+  (junction (at 123.444 107.696) (diameter 0) (color 0 0 0 0)
+  )
+  (junction (at 97.282 47.244) (diameter 0) (color 0 0 0 0)
+  )
+  (junction (at 134.239 85.217) (diameter 0) (color 0 0 0 0)
+  )
+  (junction (at 74.422 81.661) (diameter 0) (color 0 0 0 0)
+  )
+  (junction (at 144.399 108.204) (diameter 0) (color 0 0 0 0)
+  )
+  (junction (at 173.355 56.642) (diameter 0) (color 0 0 0 0)
+  )
   (junction (at 144.018 66.802) (diameter 0) (color 0 0 0 0)
   )
-  (junction (at 60.706 81.661) (diameter 0) (color 0 0 0 0)
-  )
-  (junction (at 74.549 89.027) (diameter 0) (color 0 0 0 0)
-  )
-  (junction (at 88.646 56.134) (diameter 0) (color 0 0 0 0)
-  )
-  (junction (at 220.726 48.387) (diameter 0) (color 0 0 0 0)
-  )
-  (junction (at 189.611 113.03) (diameter 0) (color 0 0 0 0)
-  )
-  (junction (at 249.555 48.387) (diameter 0) (color 0 0 0 0)
-  )
-  (junction (at 88.646 47.244) (diameter 0) (color 0 0 0 0)
-  )
-  (junction (at 240.919 66.802) (diameter 0) (color 0 0 0 0)
-  )
-  (junction (at 128.524 66.802) (diameter 0) (color 0 0 0 0)
-  )
-  (junction (at 74.549 99.314) (diameter 0) (color 0 0 0 0)
-  )
-  (junction (at 123.444 107.696) (diameter 0) (color 0 0 0 0)
-  )
-  (junction (at 97.282 47.244) (diameter 0) (color 0 0 0 0)
-  )
-  (junction (at 134.239 85.217) (diameter 0) (color 0 0 0 0)
-  )
-  (junction (at 74.422 81.661) (diameter 0) (color 0 0 0 0)
-  )
-  (junction (at 144.399 108.204) (diameter 0) (color 0 0 0 0)
-  )
-  (junction (at 173.355 56.642) (diameter 0) (color 0 0 0 0)
-  )
   (junction (at 191.77 108.458) (diameter 0) (color 0 0 0 0)
   )
@@
     (stroke (width 0) (type default) (color 0 0 0 0))
   )
+  (wire (pts (xy 161.036 113.03) (xy 161.036 114.808))
+    (stroke (width 0) (type default) (color 0 0 0 0))
+  )
+  (wire (pts (xy 249.555 48.387) (xy 249.555 49.149))
+    (stroke (width 0) (type default) (color 0 0 0 0))
+  )
+  (wire (pts (xy 102.87 80.137) (xy 102.87 67.056))
+    (stroke (width 0) (type default) (color 0 0 0 0))
+  )
+  (wire (pts (xy 189.611 108.458) (xy 189.611 113.03))
+    (stroke (width 0) (type default) (color 0 0 0 0))
+  )
+  (wire (pts (xy 62.611 85.725) (xy 60.706 85.725))
+    (stroke (width 0) (type default) (color 0 0 0 0))
+  )
+  (wire (pts (xy 230.886 78.232) (xy 197.104 78.232))
+    (stroke (width 0) (type default) (color 0 0 0 0))
+  )
+  (wire (pts (xy 137.668 108.204) (xy 144.018 108.204))
+    (stroke (width 0) (type default) (color 0 0 0 0))
+  )
+  (wire (pts (xy 60.706 81.661) (xy 62.738 81.661))
+    (stroke (width 0) (type default) (color 0 0 0 0))
+  )
+  (wire (pts (xy 137.668 119.761) (xy 137.668 117.475))
+    (stroke (width 0) (type default) (color 0 0 0 0))
+  )
+  (wire (pts (xy 102.87 100.457) (xy 102.87 101.981))
+    (stroke (width 0) (type default) (color 0 0 0 0))
+  )
+  (wire (pts (xy 220.726 49.149) (xy 220.726 48.387))
+    (stroke (width 0) (type default) (color 0 0 0 0))
+  )
+  (wire (pts (xy 207.772 48.387) (xy 207.772 49.149))
+    (stroke (width 0) (type default) (color 0 0 0 0))
+  )
+  (wire (pts (xy 147.701 56.642) (xy 139.827 56.642))
+    (stroke (width 0) (type default) (color 0 0 0 0))
+  )
+  (wire (pts (xy 58.547 81.661) (xy 59.436 81.661))
+    (stroke (width 0) (type default) (color 0 0 0 0))
+  )
+  (wire (pts (xy 74.549 98.425) (xy 74.549 99.314))
+    (stroke (width 0) (type default) (color 0 0 0 0))
+  )
+  (wire (pts (xy 191.77 108.458) (xy 192.913 108.458))
+    (stroke (width 0) (type default) (color 0 0 0 0))
+  )
+  (wire (pts (xy 144.399 116.967) (xy 144.399 119.761))
+    (stroke (width 0) (type default) (color 0 0 0 0))
+  )
+  (wire (pts (xy 233.807 48.387) (xy 240.919 48.387))
+    (stroke (width 0) (type default) (color 0 0 0 0))
+  )
+  (wire (pts (xy 173.355 48.387) (xy 173.355 56.642))
+    (stroke (width 0) (type default) (color 0 0 0 0))
+  )
+  (wire (pts (xy 90.17 95.377) (xy 85.852 95.377))
+    (stroke (width 0) (type default) (color 0 0 0 0))
+  )
+  (wire (pts (xy 117.348 66.802) (xy 128.524 66.802))
+    (stroke (width 0) (type default) (color 0 0 0 0))
+  )
   (wire (pts (xy 144.018 66.802) (xy 147.701 66.802))
-    (stroke (width 0) (type default) (color 0 0 0 0))
-  )
-  (wire (pts (xy 161.036 113.03) (xy 161.036 114.808))
-    (stroke (width 0) (type default) (color 0 0 0 0))
-  )
-  (wire (pts (xy 249.555 48.387) (xy 249.555 49.149))
-    (stroke (width 0) (type default) (color 0 0 0 0))
-  )
-  (wire (pts (xy 102.87 80.137) (xy 102.87 67.056))
-    (stroke (width 0) (type default) (color 0 0 0 0))
-  )
-  (wire (pts (xy 189.611 108.458) (xy 189.611 113.03))
-    (stroke (width 0) (type default) (color 0 0 0 0))
-  )
-  (wire (pts (xy 62.611 85.725) (xy 60.706 85.725))
-    (stroke (width 0) (type default) (color 0 0 0 0))
-  )
-  (wire (pts (xy 230.886 78.232) (xy 197.104 78.232))
-    (stroke (width 0) (type default) (color 0 0 0 0))
-  )
-  (wire (pts (xy 137.668 108.204) (xy 144.018 108.204))
-    (stroke (width 0) (type default) (color 0 0 0 0))
-  )
-  (wire (pts (xy 60.706 81.661) (xy 62.738 81.661))
-    (stroke (width 0) (type default) (color 0 0 0 0))
-  )
-  (wire (pts (xy 137.668 119.761) (xy 137.668 117.475))
-    (stroke (width 0) (type default) (color 0 0 0 0))
-  )
-  (wire (pts (xy 102.87 100.457) (xy 102.87 101.981))
-    (stroke (width 0) (type default) (color 0 0 0 0))
-  )
-  (wire (pts (xy 220.726 49.149) (xy 220.726 48.387))
-    (stroke (width 0) (type default) (color 0 0 0 0))
-  )
-  (wire (pts (xy 207.772 48.387) (xy 207.772 49.149))
-    (stroke (width 0) (type default) (color 0 0 0 0))
-  )
-  (wire (pts (xy 147.701 56.642) (xy 139.827 56.642))
-    (stroke (width 0) (type default) (color 0 0 0 0))
-  )
-  (wire (pts (xy 58.547 81.661) (xy 59.436 81.661))
-    (stroke (width 0) (type default) (color 0 0 0 0))
-  )
-  (wire (pts (xy 74.549 98.425) (xy 74.549 99.314))
-    (stroke (width 0) (type default) (color 0 0 0 0))
-  )
-  (wire (pts (xy 191.77 108.458) (xy 192.913 108.458))
-    (stroke (width 0) (type default) (color 0 0 0 0))
-  )
-  (wire (pts (xy 144.399 116.967) (xy 144.399 119.761))
-    (stroke (width 0) (type default) (color 0 0 0 0))
-  )
-  (wire (pts (xy 233.807 48.387) (xy 240.919 48.387))
-    (stroke (width 0) (type default) (color 0 0 0 0))
-  )
-  (wire (pts (xy 173.355 48.387) (xy 173.355 56.642))
-    (stroke (width 0) (type default) (color 0 0 0 0))
-  )
-  (wire (pts (xy 90.17 95.377) (xy 85.852 95.377))
-    (stroke (width 0) (type default) (color 0 0 0 0))
-  )
-  (wire (pts (xy 117.348 66.802) (xy 128.524 66.802))
     (stroke (width 0) (type default) (color 0 0 0 0))
   )
@@
     (property "Reference" "U2" (id 0) (at 175.387 101.6 0))
     (property "Value" "4N25" (id 1) (at 175.387 104.14 0))
-    (property "Footprint" "Package_DIP:DIP-6_W7.62mm" (id 2) (at 180.467 115.57 0)
+    (property "Footprint" "Package_DIP:DIP-6_W7.62mm_SMDSocket_SmallPads" (id 2) (at 180.467 115.57 0)
       (effects (font (size 1.27 1.27) italic) (justify left) hide)
     )
@@
     )
     (path "/96bdd967-f0aa-4e53-8f7d-84518c82a9df"
-      (reference "U2") (unit 1) (value "4N25") (footprint "Package_DIP:DIP-6_W7.62mm")
+      (reference "U2") (unit 1) (value "4N25") (footprint "Package_DIP:DIP-6_W7.62mm_SMDSocket_SmallPads")
     )
     (path "/b6d06dc6-d928-4921-9359-51da525bfb4e"
